File: Schematic/TunerVCO_STM32.kicad_sch (KiCad schematic)
At the start: 82 parts, among them J101 1V/OCT, J102 FM, J103 HARD SYNC, J104 SOFT SYNC, J105 PWM, J106 Pulse, J107 Saw, J108 Triangle, J109 POWER, J110 SWI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

Commit message: NeoPixel Timer/DMA stuff
Connections:
- net PIXEL: now also U104.13 (PA6); no longer U104.12 (PA5)
Changed lines of the file:
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@@
   (junction (at 155.956 250.063) (diameter 0) (color 0 0 0 0)
-  )
-  (junction (at 282.956 231.521) (diameter 0) (color 0 0 0 0)
   )
   (junction (at 233.172 35.052) (diameter 0) (color 0 0 0 0)
@@
   (no_connect (at 95.377 65.913))
   (no_connect (at 226.314 231.521))
-  (no_connect (at 266.954 234.061))
   (no_connect (at 425.958 104.521))
   (no_connect (at 266.954 241.681))
@@
   (no_connect (at 266.954 226.441))
   (no_connect (at 303.022 254))
+  (no_connect (at 266.954 231.521))
   (no_connect (at 226.314 226.441))
   (no_connect (at 266.954 239.141))
@@
     (stroke (width 0) (type default))
   )
-  (wire (pts (xy 282.956 254) (xy 282.956 231.521))
+  (wire (pts (xy 282.956 254) (xy 282.956 234.061))
     (stroke (width 0) (type default))
   )
@@
     (stroke (width 0) (type default))
   )
+  (wire (pts (xy 266.954 234.061) (xy 282.956 234.061))
+    (stroke (width 0) (type default))
+  )
   (wire (pts (xy 91.821 147.701) (xy 91.821 157.861))
     (stroke (width 0) (type default))
@@
     (stroke (width 0) (type default))
   )
-  (wire (pts (xy 266.954 231.521) (xy 282.956 231.521))
-    (stroke (width 0) (type default))
-  )
   (wire (pts (xy 361.823 112.014) (xy 361.823 110.744))
     (stroke (width 0) (type default))
@@
   )
   (wire (pts (xy 233.553 87.884) (xy 234.823 87.884))
-    (stroke (width 0) (type default))
-  )
-  (wire (pts (xy 282.956 231.521) (xy 285.496 231.521))
     (stroke (width 0) (type default))
   )
@@
     (effects (font (size 1.27 1.27)) (justify left bottom))
   )
-  (global_label "PIXEL" (shape input) (at 285.496 231.521 0) (fields_autoplaced)
+  (global_label "PIXEL" (shape input) (at 282.956 234.061 0) (fields_autoplaced)
     (effects (font (size 1.27 1.27)) (justify left))
-    (property "Intersheetrefs" "${INTERSHEET_REFS}" (at 293.7426 231.521 0)
+    (property "Intersheetrefs" "${INTERSHEET_REFS}" (at 291.2026 234.061 0)
       (effects (font (size 1.27 1.27)) (justify left) hide)
     )
